Commit message: add new controller

File: catkin_ws/src/orange_description/urdf/orange.urdf (robot description, URDF)
Before this commit: robot cool5000_description, 5 links, 4 joints
Joints:
- removed joint elbow
- removed joint shoulder
- added joint pan: type revolute, parent fixed_link, child homerus, origin xyz=0.065 0 0 rpy=0 0 0, axis 0 0 1, limit lower=-1.57 upper=1.57 effort=100 velocity=0.5
- added joint tilt: type revolute, parent homerus, child forearm, origin xyz=0.100 0 0 rpy=0 0 0, axis 0 0 1, limit lower=-1.57 upper=1.57 effort=100 velocity=0.5
